File: Extra_IO.kicad_sch (KiCad schematic)
At the start: 7 parts, among them U3 DRV2605LDGS

Commit message: Continued work, intial schematic finished
Parts:
- R9: footprint (none) -> PCM_JLCPCB:R_0603
Other:
- moved on the sheet: R9, TP1
Changed lines of the file:
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@@
 	)
 	(junction
-		(at 62.23 85.09)
+		(at 58.42 85.09)
 		(diameter 0)
 		(color 0 0 0 0)
@@
 	(wire
 		(pts
-			(xy 62.23 85.09) (xy 86.36 85.09)
-		)
-		(stroke
-			(width 0)
-			(type default)
-		)
-	)
-	(wire
-		(pts
 			(xy 111.76 80.01) (xy 116.84 80.01)
 		)
@@
 	(wire
 		(pts
+			(xy 58.42 85.09) (xy 86.36 85.09)
+		)
+		(stroke
+			(width 0)
+			(type default)
+		)
+	)
+	(wire
+		(pts
 			(xy 73.66 77.47) (xy 86.36 77.47)
+		)
+		(stroke
+			(width 0)
+			(type default)
+		)
+	)
+	(wire
+		(pts
+			(xy 57.15 85.09) (xy 58.42 85.09)
 		)
 		(stroke
@@
 	(symbol
 		(lib_id "power:GND")
-		(at 62.23 92.71 0)
+		(at 58.42 92.71 0)
 		(unit 1)
 		(exclude_from_sim no)
@@
 		(fields_autoplaced yes)
 		(property "Reference" "#PWR037"
-			(at 62.23 99.06 0)
+			(at 58.42 99.06 0)
 			(effects
 				(font
@@
 		)
 		(property "Value" "GND"
-			(at 62.23 97.79 0)
-			(effects
-				(font
-					(size 1.27 1.27)
-				)
+			(at 58.42 97.79 0)
+			(effects
+				(font
+					(size 1.27 1.27)
+				)
+				(hide yes)
 			)
 		)
 		(property "Footprint" ""
-			(at 62.23 92.71 0)
+			(at 58.42 92.71 0)
 			(effects
 				(font
@@
 		)
 		(property "Datasheet" ""
-			(at 62.23 92.71 0)
+			(at 58.42 92.71 0)
 			(effects
 				(font
@@
 		)
 		(property "Description" "Power symbol creates a global label with name \"GND\" , ground"
-			(at 62.23 92.71 0)
+			(at 58.42 92.71 0)
 			(effects
 				(font
@@
 					(size 1.27 1.27)
 				)
+				(hide yes)
 			)
 		)
@@
 	(symbol
 		(lib_id "Connector:TestPoint")
-		(at 62.23 85.09 90)
+		(at 57.15 85.09 90)
 		(unit 1)
 		(exclude_from_sim no)
@@
 		(fields_autoplaced yes)
 		(property "Reference" "TP1"
-			(at 58.928 80.01 90)
+			(at 53.848 80.01 90)
 			(effects
 				(font
@@
 		)
 		(property "Value" "TestPoint"
-			(at 58.928 82.55 90)
+			(at 53.848 82.55 90)
 			(effects
 				(font
@@
 		)
 		(property "Footprint" ""
-			(at 62.23 80.01 0)
+			(at 57.15 80.01 0)
 			(effects
 				(font
@@
 		)
 		(property "Datasheet" "~"
-			(at 62.23 80.01 0)
+			(at 57.15 80.01 0)
 			(effects
 				(font
@@
 		)
 		(property "Description" "test point"
-			(at 62.23 85.09 0)
+			(at 57.15 85.09 0)
 			(effects
 				(font
@@
 					(size 1.27 1.27)
 				)
+				(hide yes)
 			)
 		)
@@
 					(size 1.27 1.27)
 				)
+				(hide yes)
 			)
 		)
@@
 	(symbol
 		(lib_id "Device:R")
-		(at 62.23 88.9 180)
+		(at 58.42 88.9 180)
 		(unit 1)
 		(exclude_from_sim no)
@@
 		(fields_autoplaced yes)
 		(property "Reference" "R9"
-			(at 64.77 87.6299 0)
+			(at 60.96 87.6299 0)
 			(effects
 				(font
@@
 		)
 		(property "Value" "10k"
-			(at 64.77 90.1699 0)
+			(at 60.96 90.1699 0)
 			(effects
 				(font
@@
 			)
 		)
-		(property "Footprint" ""
-			(at 64.008 88.9 90)
+		(property "Footprint" "PCM_JLCPCB:R_0603"
+			(at 60.198 88.9 90)
 			(effects
 				(font
@@
 		)
 		(property "Datasheet" "~"
-			(at 62.23 88.9 0)
+			(at 58.42 88.9 0)
 			(effects
 				(font
@@
 		)
 		(property "Description" "Resistor"
-			(at 62.23 88.9 0)
-			(effects
-				(font
+			(at 58.42 88.9 0)
+			(effects
+				(font
