File: MCU.kicad_sch (KiCad schematic)
At the start: 17 parts, among them J2 3221-10-0100-00, SW1 SW_DPST_x2, SW2 SW_DPST_x2, SW3 SW_DPST_x2, SW4 SW_DPST_x2, SW5 SW_DPST_x2, SW6 SW_DPST_x2, SW7 SW_DPST_x2, U4 BGM220PC22HNA2, U6 DRV5053CAQDBZR

Commit message: Continued work, intial schematic finished
Parts:
- added R14, R15: 10k, PCM_JLCPCB:R_0603, symbol Device:R
- added R16, R17: DNP, PCM_JLCPCB:R_0603, symbol Device:R
- R1, R10, R11, R2: footprint (none) -> PCM_JLCPCB:R_0603
Connections:
- net +3V3: now also R16.2, R17.2
- net GND: now also R14.1, R15.1
- net Board_ID_1: now reaches U4.18 (PD03)
- net Board_ID_1: now also R15.2, R17.1
- net Board_ID_0: now reaches U4.19 (PD02)
- net Board_ID_0: now also R14.2, R16.1
Other:
- moved on the sheet: J2, R10, R11, U6
