File: Power.kicad_sch (KiCad schematic)
At the start: 19 parts, among them J1 B2B-PH-K-S, U1 BQ24075RGT, U2 TPS63031DSK, U5 MAX17048G_T10

Commit message: Continued work, intial schematic finished
Parts:
- added R12: OR, PCM_JLCPCB:R_0603, symbol Device:R
- added R13: DNP, PCM_JLCPCB:R_0603, symbol Device:R
- added TP2: 3v3_VIN_REG, symbol Connector:TestPoint
- added TP3: TestPoint, symbol Connector:TestPoint
- R3, R4, R5, R6, R7, R8: footprint (none) -> PCM_JLCPCB:R_0603
Connections:
- net +3V3: now also TP3.1
- net +5V: now also R13.2
- net VBUS: now also R12.2; no longer C4.1, U2.5 (VIN)
- new net: C4.1, R12.1, R13.1, TP2.1, U2.5 (VIN)
