File: handheld_hardware.kicad_pcb (KiCad board)
At the start: 2 copper layers, 4 parts, among them U1 BQ24075RGT, U2 TPS63031DSK, U3 DRV2605LDGS, U4 BGM220PC22HNA2

Commit message: Continued work, intial schematic finished
Parts:
- added R1: 2.2k, PCM_JLCPCB:R_0603, F.Cu at (166.6, 102.5)
- added R10: 0R, PCM_JLCPCB:R_0603, F.Cu at (166.6, 107.0)
- added R11: 0R, PCM_JLCPCB:R_0603, F.Cu at (166.6, 109.2)
- added R12: OR, PCM_JLCPCB:R_0603, F.Cu at (161.0, 116.0)
- added R13: DNP, PCM_JLCPCB:R_0603, F.Cu at (163.7, 122.4)
- added R14: 10k, PCM_JLCPCB:R_0603, F.Cu at (166.6, 111.5)
- added R15: 10k, PCM_JLCPCB:R_0603, F.Cu at (166.6, 113.8)
- added R16: DNP, PCM_JLCPCB:R_0603, F.Cu at (172.4, 117.3)
- added R17: DNP, PCM_JLCPCB:R_0603, F.Cu at (169.4, 122.4)
- added R2: 2.2k, PCM_JLCPCB:R_0603, F.Cu at (166.6, 104.8)
- added R3: 10k, PCM_JLCPCB:R_0603, F.Cu at (161.0, 102.5)
- added R4: 10k, PCM_JLCPCB:R_0603, F.Cu at (161.0, 104.8)
- added R5: 1.18k?, PCM_JLCPCB:R_0603, F.Cu at (161.0, 107.0)
- added R6: 1.13k?, PCM_JLCPCB:R_0603, F.Cu at (161.0, 109.2)
- added R7: 10k, PCM_JLCPCB:R_0603, F.Cu at (161.0, 111.5)
- added R8: 10k, PCM_JLCPCB:R_0603, F.Cu at (161.0, 113.8)
- added R9: 10k, PCM_JLCPCB:R_0603, F.Cu at (172.3, 102.5)
- added U5: MAX17048G_T10, MAX17048G_T10:SON50P200X200X80-9N, F.Cu at (120.2, 104.0)
- added U6: DRV5053CAQDBZR, DRV5053CAQDBZR:SOT95P237X112-3N, F.Cu at (133.0, 114.0)
- added VR1: RKJXV1224005, RKJXV1224005:RKJXV1224005, F.Cu at (127.5, 126.5)
- moved U4 6.64 mm to (112.6, 79.3)
Connections:
- U2 pad 5: VBUS -> Net-(U2-VIN)
- U4 pad 18: unconnected-(U4-PD03-Pad18) -> /MCU/Board_ID_1
- U4 pad 19: unconnected-(U4-PD02-Pad19) -> /MCU/Board_ID_0
