File: handheld_hardware.kicad_sch (KiCad schematic)
At the start: 0 parts

Commit message: Continued work, intial schematic finished
Parts:
- added H1, H2, H3, H4: MountingHole, symbol Mechanical:MountingHole
